Commit message: bwh ros control + description

File: galil_description/urdf/galil.xacro (robot description, xacro)
@@ -2,71 +2,58 @@
 <robot xmlns:xacro="http://wiki.ros.org/xacro">
   <xacro:macro name="galil">
-    <!-- links -  main serial chain -->
-    <link name="base_link"/>
-    <link name="insertion_link">
+    <xacro:include filename="$(find galil_description)/urdf/materials.xacro" />
+    <link name="base_link">
       <visual>
-        <origin xyz="0 0 0" rpy="0 0 ${pi}"/>
-        <geometry>
-          <box size="1 1 1"/>
+	<origin xyz="0 0 0" rpy="0 0 0"/>
+	<geometry>
+	  <mesh filename="package://galil_description/meshes/base_link.stl"/>
 	</geometry>
+	<material name="silver"/>
       </visual>
-      <collision>
-        <origin xyz="0 0 0" rpy="0 0 ${pi}"/>
-        <geometry>
-          <box size="1 1 1"/>
-        </geometry>
-      </collision>
+    </link>
+    <link name="needle_link">
+      <visual>
+	<geometry>
+	  <mesh filename="package://galil_description/meshes/needle_link.stl"/>
+	</geometry>
+	<material name="silver"/>
+      </visual>
+    </link>
+    <link name="vertical_link">
+      <visual>
+	<geometry>
+	  <mesh filename="package://galil_description/meshes/vertical_link.stl"/>
+	</geometry>
+	<material name="silver"/>
+      </visual>
+    </link>
+    <link name="horizontal_link">
+      <visual>
+	<geometry>
+	  <mesh filename="package://galil_description/meshes/horizontal_link.stl"/>
+	</geometry>
+	<material name="silver"/>
+      </visual>
     </link>
     <joint name="insertion_joint" type="prismatic">
-      <origin xyz="0 0 0" rpy="0 0 0" />
-      <axis xyz="0 0 1" />
-      <parent link="base_link" />
-      <child link="insertion_link" />
-      <limit lower="0" upper="100"
-             effort="100" velocity="10"/>
+      <origin xyz="0 0 0" rpy="0 0 0"/>
+      <parent link="horizontal_link"/>
+      <child link="needle_link"/>
+      <axis xyz="-1.0 0.0 0.0"/>
+      <limit upper="0.1" lower="0.0" effort="100" velocity="100"/>
     </joint>
-    <link name="template_horizontal">
-      <visual>
-        <origin xyz="0 0 0" rpy="0 0 0"/>
-        <geometry>
-          <box size="1 1 1"/>
-	</geometry>
-      </visual>
-      <collision>
-        <origin xyz="0 0 0" rpy="0 0 0"/>
-        <geometry>
-          <box size="1 1 1"/>
-        </geometry>
-      </collision>
-    </link>
-    <joint name="template_horizontal_joint" type="prismatic">
-      <origin xyz="0 0 0" rpy="0 0 0" />
-      <axis xyz="0 0 1" />
-      <parent link="base_link" />
-      <child link="template_horizontal_link" />
-      <limit lower="0" upper="100"
-             effort="100" velocity="10"/>
+    <joint name="horizontal_joint" type="prismatic">
+      <origin xyz="0 0 0" rpy="0 0 0"/>
+      <parent link="vertical_link"/>
+      <child link="horizontal_link"/>
+      <axis xyz="0.0 1.0 0.0"/>
+      <limit upper="0.03" lower="-0.03" effort="100" velocity="100"/>
     </joint>
-    <link name="template_verticalal">
-      <visual>
-        <origin xyz="0 0 0" rpy="0 0 0"/>
-        <geometry>
-          <box size="1 1 1"/>
-	</geometry>
-      </visual>
-      <collision>
-        <origin xyz="0 0 0" rpy="0 0 0"/>
-        <geometry>
-          <box size="1 1 1"/>
-        </geometry>
-      </collision>
-    </link>
-    <joint name="template_vertical_joint" type="prismatic">
-      <origin xyz="0 0 0" rpy="0 0 0" />
-      <axis xyz="0 0 1" />
-      <parent link="template_horizontal_link" />
-      <child link="template_vertical_link" />
-      <limit lower="0" upper="100"
-             effort="100" velocity="10"/>
+    <joint name="vertical_joint" type="prismatic">
+      <origin xyz="0 0 0" rpy="0 0 0"/>
+      <parent link="base_link"/>
+      <child link="vertical_link"/>
+      <axis xyz="0.0 0.0 1.0"/>
+      <limit upper="0.05" lower="0.0" effort="100" velocity="100"/>
     </joint>
   </xacro:macro>
